File: pcb/Luciebox/_autosave-R2-R_ladder_dac.sch (KiCad schematic (older format))
At the start: 25 parts, among them T2 terminal_8x1

Commit message: pcb progress'
Changed lines of the file:
@@
 AR Path="/5D761BCA/5D7526B9" Ref="R52"  Part="1"
 AR Path="/5D9307E8/5D7526B9" Ref="R76"  Part="1"
-F 0 "R76" H 2609 3596 50  0000 L CNN
+F 0 "R28" H 2609 3596 50  0000 L CNN
 F 1 "R_Small" H 2609 3505 50  0000 L CNN
 F 2 "Luciebox:1206" H 2550 3550 50  0001 C CNN
@@
 AR Path="/5D761BCA/5D7526BF" Ref="R67"  Part="1"
 AR Path="/5D9307E8/5D7526BF" Ref="R91"  Part="1"
-F 0 "R91" H 2609 3896 50  0000 L CNN
+F 0 "R43" H 2609 3896 50  0000 L CNN
 F 1 "R_Small" H 2609 3805 50  0000 L CNN
 F 2 "Luciebox:1206" H 2550 3850 50  0001 C CNN
@@
 AR Path="/5D761BCA/5D7526C5" Ref="R60"  Part="1"
 AR Path="/5D9307E8/5D7526C5" Ref="R84"  Part="1"
-F 0 "R84" H 2759 3746 50  0000 L CNN
+F 0 "R36" H 2759 3746 50  0000 L CNN
 F 1 "R_Small" H 2759 3655 50  0000 L CNN
 F 2 "Luciebox:1206" H 2700 3700 50  0001 C CNN
@@
 AR Path="/5D761BCA/5D7526CF" Ref="R51"  Part="1"
 AR Path="/5D9307E8/5D7526CF" Ref="R75"  Part="1"
-F 0 "R75" H 3709 2246 50  0000 L CNN
+F 0 "R27" H 3709 2246 50  0000 L CNN
 F 1 "R_Small" H 3709 2155 50  0000 L CNN
 F 2 "Luciebox:1206" H 3650 2200 50  0001 C CNN
@@
 AR Path="/5D761BCA/5D7526D5" Ref="T3"  Part="1"
 AR Path="/5D9307E8/5D7526D5" Ref="T4"  Part="1"
-F 0 "T4" V 3765 3650 50  0000 C CNN
+F 0 "T2" V 3765 3650 50  0000 C CNN
 F 1 "terminal_8x1" V 3674 3650 50  0000 C CNN
 F 2 "Luciebox:Terminal_8x1_100mil" H 3250 3050 50  0001 C CNN
@@
 AR Path="/5D761BCA/5D7526DB" Ref="R50"  Part="1"
 AR Path="/5D9307E8/5D7526DB" Ref="R74"  Part="1"
-F 0 "R74" H 3559 2246 50  0000 L CNN
+F 0 "R26" H 3559 2246 50  0000 L CNN
 F 1 "R_Small" H 3559 2155 50  0000 L CNN
 F 2 "Luciebox:1206" H 3500 2200 50  0001 C CNN
@@
 AR Path="/5D761BCA/5D7526E1" Ref="R49"  Part="1"
 AR Path="/5D9307E8/5D7526E1" Ref="R73"  Part="1"
-F 0 "R73" H 3409 2246 50  0000 L CNN
+F 0 "R25" H 3409 2246 50  0000 L CNN
 F 1 "R_Small" H 3409 2155 50  0000 L CNN
 F 2 "Luciebox:1206" H 3350 2200 50  0001 C CNN
@@
 AR Path="/5D761BCA/5D7526E7" Ref="R48"  Part="1"
 AR Path="/5D9307E8/5D7526E7" Ref="R72"  Part="1"
-F 0 "R72" H 3259 2246 50  0000 L CNN
+F 0 "R24" H 3259 2246 50  0000 L CNN
 F 1 "R_Small" H 3259 2155 50  0000 L CNN
 F 2 "Luciebox:1206" H 3200 2200 50  0001 C CNN
@@
 AR Path="/5D761BCA/5D7526ED" Ref="R47"  Part="1"
 AR Path="/5D9307E8/5D7526ED" Ref="R71"  Part="1"
-F 0 "R71" H 3109 2246 50  0000 L CNN
+F 0 "R23" H 3109 2246 50  0000 L CNN
 F 1 "R_Small" H 3109 2155 50  0000 L CNN
 F 2 "Luciebox:1206" H 3050 2200 50  0001 C CNN
@@
 AR Path="/5D761BCA/5D7526F3" Ref="R46"  Part="1"
 AR Path="/5D9307E8/5D7526F3" Ref="R70"  Part="1"
-F 0 "R70" H 2959 2246 50  0000 L CNN
+F 0 "R22" H 2959 2246 50  0000 L CNN
 F 1 "R_Small" H 2959 2155 50  0000 L CNN
 F 2 "Luciebox:1206" H 2900 2200 50  0001 C CNN
@@
 AR Path="/5D761BCA/5D7526F9" Ref="R45"  Part="1"
 AR Path="/5D9307E8/5D7526F9" Ref="R69"  Part="1"
-F 0 "R69" H 2809 2246 50  0000 L CNN
+F 0 "R21" H 2809 2246 50  0000 L CNN
 F 1 "R_Small" H 2809 2155 50  0000 L CNN
 F 2 "Luciebox:1206" H 2750 2200 50  0001 C CNN
@@
 AR Path="/5D761BCA/5D7526FF" Ref="R53"  Part="1"
 AR Path="/5D9307E8/5D7526FF" Ref="R77"  Part="1"
-F 0 "R77" H 2909 3596 50  0000 L CNN
+F 0 "R29" H 2909 3596 50  0000 L CNN
 F 1 "R_Small" H 2909 3505 50  0000 L CNN
 F 2 "Luciebox:1206" H 2850 3550 50  0001 C CNN
@@
 AR Path="/5D761BCA/5D752705" Ref="R61"  Part="1"
 AR Path="/5D9307E8/5D752705" Ref="R85"  Part="1"
-F 0 "R85" H 3059 3746 50  0000 L CNN
+F 0 "R37" H 3059 3746 50  0000 L CNN
 F 1 "R_Small" H 3059 3655 50  0000 L CNN
 F 2 "Luciebox:1206" H 3000 3700 50  0001 C CNN
@@
 AR Path="/5D761BCA/5D75270D" Ref="R54"  Part="1"
 AR Path="/5D9307E8/5D75270D" Ref="R78"  Part="1"
-F 0 "R78" H 3209 3596 50  0000 L CNN
+F 0 "R30" H 3209 3596 50  0000 L CNN
 F 1 "R_Small" H 3209 3505 50  0000 L CNN
 F 2 "Luciebox:1206" H 3150 3550 50  0001 C CNN
@@
 AR Path="/5D761BCA/5D752715" Ref="R62"  Part="1"
 AR Path="/5D9307E8/5D752715" Ref="R86"  Part="1"
-F 0 "R86" H 3359 3746 50  0000 L CNN
+F 0 "R38" H 3359 3746 50  0000 L CNN
 F 1 "R_Small" H 3359 3655 50  0000 L CNN
 F 2 "Luciebox:1206" H 3300 3700 50  0001 C CNN
@@
 AR Path="/5D761BCA/5D75271B" Ref="R63"  Part="1"
 AR Path="/5D9307E8/5D75271B" Ref="R87"  Part="1"
-F 0 "R87" H 3659 3746 50  0000 L CNN
+F 0 "R39" H 3659 3746 50  0000 L CNN
 F 1 "R_Small" H 3659 3655 50  0000 L CNN
 F 2 "Luciebox:1206" H 3600 3700 50  0001 C CNN
@@
 AR Path="/5D761BCA/5D752721" Ref="R55"  Part="1"
 AR Path="/5D9307E8/5D752721" Ref="R79"  Part="1"
-F 0 "R79" H 3509 3596 50  0000 L CNN
+F 0 "R31" H 3509 3596 50  0000 L CNN
 F 1 "R_Small" H 3509 3505 50  0000 L CNN
 F 2 "Luciebox:1206" H 3450 3550 50  0001 C CNN
@@
 AR Path="/5D761BCA/5D752727" Ref="R56"  Part="1"
 AR Path="/5D9307E8/5D752727" Ref="R80"  Part="1"
-F 0 "R80" H 3809 3596 50  0000 L CNN
+F 0 "R32" H 3809 3596 50  0000 L CNN
 F 1 "R_Small" H 3809 3505 50  0000 L CNN
 F 2 "Luciebox:1206" H 3750 3550 50  0001 C CNN
@@
 AR Path="/5D761BCA/5D75272D" Ref="R64"  Part="1"
 AR Path="/5D9307E8/5D75272D" Ref="R88"  Part="1"
-F 0 "R88" H 3959 3746 50  0000 L CNN
+F 0 "R40" H 3959 3746 50  0000 L CNN
 F 1 "R_Small" H 3959 3655 50  0000 L CNN
 F 2 "Luciebox:1206" H 3900 3700 50  0001 C CNN
@@
 AR Path="/5D761BCA/5D75273F" Ref="R57"  Part="1"
 AR Path="/5D9307E8/5D75273F" Ref="R81"  Part="1"
-F 0 "R81" H 4109 3596 50  0000 L CNN
+F 0 "R33" H 4109 3596 50  0000 L CNN
 F 1 "R_Small" H 4109 3505 50  0000 L CNN
 F 2 "Luciebox:1206" H 4050 3550 50  0001 C CNN
@@
 AR Path="/5D761BCA/5D752745" Ref="R65"  Part="1"
 AR Path="/5D9307E8/5D752745" Ref="R89"  Part="1"
-F 0 "R89" H 4259 3746 50  0000 L CNN
+F 0 "R41" H 4259 3746 50  0000 L CNN
 F 1 "R_Small" H 4259 3655 50  0000 L CNN
 F 2 "Luciebox:1206" H 4200 3700 50  0001 C CNN
@@
 AR Path="/5D761BCA/5D75274B" Ref="R66"  Part="1"
 AR Path="/5D9307E8/5D75274B" Ref="R90"  Part="1"
-F 0 "R90" H 4559 3746 50  0000 L CNN
+F 0 "R42" H 4559 3746 50  0000 L CNN
 F 1 "R_Small" H 4559 3655 50  0000 L CNN
 F 2 "Luciebox:1206" H 4500 3700 50  0001 C CNN
@@
 AR Path="/5D761BCA/5D752751" Ref="R58"  Part="1"
 AR Path="/5D9307E8/5D752751" Ref="R82"  Part="1"
-F 0 "R82" H 4409 3596 50  0000 L CNN
+F 0 "R34" H 4409 3596 50  0000 L CNN
 F 1 "R_Small" H 4409 3505 50  0000 L CNN
 F 2 "Luciebox:1206" H 4350 3550 50  0001 C CNN
@@
 AR Path="/5D761BCA/5D752757" Ref="R59"  Part="1"
 AR Path="/5D9307E8/5D752757" Ref="R83"  Part="1"
-F 0 "R83" H 4709 3596 50  0000 L CNN
+F 0 "R35" H 4709 3596 50  0000 L CNN
 F 1 "R_Small" H 4709 3505 50  0000 L CNN
 F 2 "Luciebox:1206" H 4650 3550 50  0001 C CNN
@@
 AR Path="/5D761BCA/5D752769" Ref="#PWR022"  Part="1"
 AR Path="/5D9307E8/5D752769" Ref="#PWR024"  Part="1"
-F 0 "#PWR024" H 2550 3700 50  0001 C CNN
+F 0 "#PWR020" H 2550 3700 50  0001 C CNN
 F 1 "GND" H 2555 3777 50  0000 C CNN
 F 2 "" H 2550 3950 50  0001 C CNN
@@
 AR Path="/5D761BCA/5D75277B" Ref="#PWR021"  Part="1"
 AR Path="/5D9307E8/5D75277B" Ref="#PWR023"  Part="1"
-F 0 "#PWR023" H 3850 1650 50  0001 C CNN
+F 0 "#PWR019" H 3850 1650 50  0001 C CNN
 F 1 "GND" H 3855 1727 50  0000 C CNN
 F 2 "" H 3850 1900 50  0001 C CNN
@@
 AR Path="/5D761BCA/5D7527B8" Ref="R44"  Part="1"
 AR Path="/5D9307E8/5D7527B8" Ref="R68"  Part="1"
-F 0 "R68" H 2659 2246 50  0000 L CNN
+F 0 "R20" H 2659 2246 50  0000 L CNN
 F 1 "R_Small" H 2659 2155 50  0000 L CNN
 F 2 "Luciebox:1206" H 2600 2200 50  0001 C CNN
