File: pcb/Luciebox/Luciebox.sch (KiCad schematic (older format))
At the start: 45 parts, among them J1 Screw_Terminal_01x07, J2 Screw_Terminal_01x07, J3 Screw_Terminal_01x07, P1 Power, P2 Analog, P3 Digital, P4 Digital, P5 CONN_01X01, P6 CONN_01X01, P7 CONN_01X01, P8 CONN_01X01, Q1 BC558, U1 CA56-12SRWA, U2 ULN2003A, U3 ATmega328-PU

Commit message: pcb progress'
Parts:
- removed R? (x24): R_Small, Luciebox:1206, symbol Device:R_Small
- removed T?: terminal_8x1, Luciebox:Terminal_8x1_100mil, symbol Luciebox_components:terminal_8x1
- added BZ1: Buzzer, Luciebox:buzzer, symbol Device:Buzzer
- added C1: 100nF, Luciebox:0805, symbol Device:C_Small
- added C2, C3: 20pF, Luciebox:0805, symbol Device:C_Small
- added J4: Screw_Terminal_01x07, Luciebox:Terminal_7x1_100mil, symbol Connector:Screw_Terminal_01x07
- added R10, R11, R12, R13, R14, R15, R16, R17, R18, R7, R8, R9: 10K, Luciebox:1206, symbol Device:R_Small
- added R19: 100, Luciebox:1206, symbol Device:R_Small
- added R6: 1M, Luciebox:1206, symbol Device:R_Small
- added RV1: R_POT, symbol Device:R_POT
- added T1: terminal_13x1, Luciebox:Terminal_13x1_100mil, symbol Luciebox_components:terminal_13x1
- added Y1: 16MHz, Luciebox:0805, symbol Device:Crystal
- J1, J2, J3: footprint Luciebox:Term_Block_1x7_P5.08mm -> Luciebox:Terminal_7x1_100mil
- R1: renamed from R5; value R_Small -> 100
- R2: renamed from R1; value R_Small -> 100
- R3: renamed from R2; value R_Small -> 100
- R4: renamed from R3; value R_Small -> 100
- R5: renamed from R4; value R_Small -> 100
- renumbered P5 to P1, P6 to P2, P7 to P3, P8 to P4, P3 to P5, P1 to P6, P4 to P7, P2 to P8
Connections:
- net 0(Rx): now also U3.2 (PD0), J4.4 (Pin_4)
- net 1(Tx): now also U3.3 (PD1), J4.3 (Pin_3)
- net 10(PWM-SS): now also U3.16 (PB2)
- net 11(PWM-MOSI): now also U3.17 (PB3)
- net 12(MISO): now also U3.18 (PB4)
- net 13(SCK): now also U3.19 (PB5)
- net 2: now also U3.4 (PD2)
- net 3(PWM): now also U3.5 (PD3)
- net 4: now also U3.6 (PD4)
- net 5(PWM): now also U3.11 (PD5)
- net 6(PWM): now also U3.12 (PD6)
- net 7: now also U3.13 (PD7)
- net 8: now also U3.14 (PB0)
- net 9(PWM): now also U3.15 (PB1)
- net A0: now also U3.23 (PC0), T1.13 (OUT)
- net A1: now also U3.24 (PC1)
- net A2: now also U3.25 (PC2)
- net A3: now also U3.26 (PC3), RV1.2
- net A4(SDA): now also U3.27 (PC4)
- net A5(SCL): now also U3.28 (PC5), BZ1.1 (-)
- net GND: now also U3.22 (GND), U3.8 (GND), BZ1.2 (+), C1.2, C2.1, C3.1, J4.2 (Pin_2), R7.2, RV1.3
- net at U3.1 (~RESET~/PC6): now also J4.5 (Pin_5), R19.2
- net at U3.10 (XTAL2/PB7): now also C3.2, R6.2, Y1.2
- net VCC: now reaches U3.20 (AVCC)
- net VCC: now also U3.21 (AREF), U3.7 (VCC), C1.1, J4.1 (Pin_1), R18.1, R19.1, RV1.1, T1.1
- net at U3.9 (XTAL1/PB6): now also C2.2, R6.1, Y1.1
- new net: R7.1, R8.2, T1.12
- new net: R8.1, R9.2, T1.11
- new net: R10.2, R9.1, T1.10
- new net: R10.1, R11.2, T1.9
- new net: R11.1, R12.2, T1.8
- new net: R12.1, R13.2, T1.7
- new net: R13.1, R14.2, T1.6
- new net: R14.1, R15.2, T1.5
- new net: R15.1, R16.2, T1.4
- new net: R16.1, R17.2, T1.3
- new net: R17.1, R18.2, T1.2

Commit message: pcb progress dedicated R-2R ladder'
Parts:
- Y1: footprint Luciebox:0805 -> (none)
Changed lines of the file:
@@
 F 0 "Y1" V 9704 4631 50  0000 L CNN
 F 1 "16MHz" V 9795 4631 50  0000 L CNN
-F 2 "Luciebox:0805" H 9750 4500 50  0001 C CNN
+F 2 "" H 9750 4500 50  0001 C CNN
 F 3 "~" H 9750 4500 50  0001 C CNN
 	1    9750 4500
