File: pcb/Luciebox/R2-R_ladder_dac_tilt_switches.sch (KiCad schematic (older format))
At the start: 9 parts, among them SW10 Switch_tilt, SW11 Switch_tilt, SW12 Switch_tilt, SW9 Switch_tilt

Commit message: progressive change towards v2.0
Parts:
- R24, R25, R26, R27: footprint Luciebox:1206 -> Luciebox:1206_0805
Changed lines of the file:
@@
 F 0 "R44" H 3809 2446 50  0000 L CNN
 F 1 "R_Small" H 3809 2355 50  0000 L CNN
-F 2 "Luciebox:1206" H 3750 2400 50  0001 C CNN
+F 2 "Luciebox:1206_0805" H 3750 2400 50  0001 C CNN
 F 3 "~" H 3750 2400 50  0001 C CNN
 	1    3750 2400
@@
 F 0 "R43" H 3809 1996 50  0000 L CNN
 F 1 "R_Small" H 3809 1905 50  0000 L CNN
-F 2 "Luciebox:1206" H 3750 1950 50  0001 C CNN
+F 2 "Luciebox:1206_0805" H 3750 1950 50  0001 C CNN
 F 3 "~" H 3750 1950 50  0001 C CNN
 	1    3750 1950
@@
 	5750 2850 5250 2850
 Wire Wire Line
-	4150 2850 4150 3500
-Wire Wire Line
-	4150 3500 3250 3500
-Wire Wire Line
-	3250 3500 3250 3700
-Wire Wire Line
-	3150 3450 4100 3450
-Wire Wire Line
-	4100 3450 4100 2400
-Wire Wire Line
-	3150 3450 3150 3700
-Wire Wire Line
-	4050 1950 4050 3400
-Wire Wire Line
-	4050 3400 3050 3400
-Wire Wire Line
-	3050 3400 3050 3700
-Wire Wire Line
-	2950 3350 4000 3350
-Wire Wire Line
-	4000 3350 4000 1500
-Wire Wire Line
-	2950 3350 2950 3700
-Wire Wire Line
 	5750 1500 5750 1950
 Wire Wire Line
@@
 F 0 "R45" H 3809 2896 50  0000 L CNN
 F 1 "R_Small" H 3809 2805 50  0000 L CNN
-F 2 "Luciebox:1206" H 3750 2850 50  0001 C CNN
+F 2 "Luciebox:1206_0805" H 3750 2850 50  0001 C CNN
 F 3 "~" H 3750 2850 50  0001 C CNN
 	1    3750 2850
@@
 F 0 "R42" H 3809 1546 50  0000 L CNN
 F 1 "R_Small" H 3809 1455 50  0000 L CNN
-F 2 "Luciebox:1206" H 3750 1500 50  0001 C CNN
+F 2 "Luciebox:1206_0805" H 3750 1500 50  0001 C CNN
 F 3 "~" H 3750 1500 50  0001 C CNN
 	1    3750 1500
 	0    -1   -1   0
 $EndComp
-Wire Wire Line
-	4000 1500 4900 1500
-Wire Wire Line
-	4150 2850 4900 2850
-Wire Wire Line
-	4100 2400 4900 2400
-Wire Wire Line
-	4050 1950 4900 1950
-Wire Wire Line
-	3850 1500 4000 1500
-Connection ~ 4000 1500
-Wire Wire Line
-	3850 1950 4050 1950
-Connection ~ 4050 1950
-Wire Wire Line
-	3850 2400 4100 2400
-Connection ~ 4100 2400
-Wire Wire Line
-	3850 2850 4150 2850
-Connection ~ 4150 2850
 Wire Wire Line
 	3650 1500 3550 1500
@@
 	3550 3000 3550 2850
 Connection ~ 3550 2850
+Wire Wire Line
+	3850 1500 4100 1500
+Wire Wire Line
+	3850 1950 4200 1950
+Wire Wire Line
+	3850 2400 4300 2400
+Wire Wire Line
+	3850 2850 4400 2850
+Wire Wire Line
+	4400 2850 4400 3500
+Wire Wire Line
+	4400 3500 3250 3500
+Wire Wire Line
+	3250 3500 3250 3700
+Connection ~ 4400 2850
+Wire Wire Line
+	4400 2850 4900 2850
+Wire Wire Line
+	3150 3700 3150 3400
+Wire Wire Line
+	3150 3400 4300 3400
+Wire Wire Line
+	4300 3400 4300 2400
+Connection ~ 4300 2400
+Wire Wire Line
+	4300 2400 4900 2400
+Wire Wire Line
+	4200 1950 4200 3300
+Wire Wire Line
+	4200 3300 3050 3300
+Wire Wire Line
+	3050 3300 3050 3700
+Connection ~ 4200 1950
+Wire Wire Line
+	4200 1950 4900 1950
+Wire Wire Line
+	2950 3700 2950 3200
+Wire Wire Line
+	2950 3200 4100 3200
+Wire Wire Line
+	4100 3200 4100 1500
+Connection ~ 4100 1500
+Wire Wire Line
+	4100 1500 4900 1500
 $EndSCHEMATC

Commit message: add holes for R-2R ladder, fix bug with tilt switch sheet. Set output led's. All good here.
Connections:
- net DAC_analog_out: now reaches R28.1
Changed lines of the file:
@@
 AR Path="/5D761BCA/5D7526DB" Ref="R35"  Part="1"
 AR Path="/5D9307E8/5D7526DB" Ref="R44"  Part="1"
+AR Path="/5EB37636/5D7526DB" Ref="R?"  Part="1"
+AR Path="/5EBCF42E/5D7526DB" Ref="R?"  Part="1"
 F 0 "R44" H 3809 2446 50  0000 L CNN
 F 1 "R_Small" H 3809 2355 50  0000 L CNN
@@
 AR Path="/5D761BCA/5D7526E1" Ref="R34"  Part="1"
 AR Path="/5D9307E8/5D7526E1" Ref="R43"  Part="1"
+AR Path="/5EB37636/5D7526E1" Ref="R?"  Part="1"
+AR Path="/5EBCF42E/5D7526E1" Ref="R?"  Part="1"
 F 0 "R43" H 3809 1996 50  0000 L CNN
 F 1 "R_Small" H 3809 1905 50  0000 L CNN
@@
 AR Path="/5D761BCA/5DABC300" Ref="R37"  Part="1"
 AR Path="/5D9307E8/5DABC300" Ref="R46"  Part="1"
+AR Path="/5EB37636/5DABC300" Ref="R?"  Part="1"
+AR Path="/5EBCF42E/5DABC300" Ref="R?"  Part="1"
 F 0 "R46" V 2746 4778 50  0000 L CNN
 F 1 "DAC_R-2R" V 2837 4778 50  0000 L CNN
@@
 AR Path="/5D761BCA/5E6454E3" Ref="#PWR024"  Part="1"
 AR Path="/5D9307E8/5E6454E3" Ref="#PWR027"  Part="1"
+AR Path="/5EB37636/5E6454E3" Ref="#PWR?"  Part="1"
+AR Path="/5EBCF42E/5E6454E3" Ref="#PWR?"  Part="1"
 F 0 "#PWR027" H 3600 3300 50  0001 C CNN
 F 1 "GND" H 3605 3377 50  0000 C CNN
@@
 AR Path="/5D74964C/5E6454E4" Ref="#PWR019"  Part="1"
 AR Path="/5D761BCA/5E6454E4" Ref="#PWR022"  Part="1"
+AR Path="/5EB37636/5E6454E4" Ref="#PWR?"  Part="1"
+AR Path="/5EBCF42E/5E6454E4" Ref="#PWR?"  Part="1"
 F 0 "#PWR025" H 5750 1350 50  0001 C CNN
 F 1 "VCC_minimalCurrent" H 5767 1673 50  0000 C CNN
@@
 AR Path="/5D74964C/5E2DD851" Ref="SW1"  Part="1"
 AR Path="/5D761BCA/5E2DD851" Ref="SW5"  Part="1"
+AR Path="/5EB37636/5E2DD851" Ref="SW?"  Part="1"
+AR Path="/5EBCF42E/5E2DD851" Ref="SW?"  Part="1"
 F 0 "SW9" H 5075 1765 50  0000 C CNN
 F 1 "Switch_tilt" H 5075 1674 50  0000 C CNN
@@
 AR Path="/5D74964C/5E2DEE2B" Ref="SW2"  Part="1"
 AR Path="/5D761BCA/5E2DEE2B" Ref="SW6"  Part="1"
+AR Path="/5EB37636/5E2DEE2B" Ref="SW?"  Part="1"
+AR Path="/5EBCF42E/5E2DEE2B" Ref="SW?"  Part="1"
 F 0 "SW10" H 5075 2215 50  0000 C CNN
 F 1 "Switch_tilt" H 5075 2124 50  0000 C CNN
@@
 AR Path="/5D74964C/5E2DF258" Ref="SW3"  Part="1"
 AR Path="/5D761BCA/5E2DF258" Ref="SW7"  Part="1"
+AR Path="/5EB37636/5E2DF258" Ref="SW?"  Part="1"
+AR Path="/5EBCF42E/5E2DF258" Ref="SW?"  Part="1"
 F 0 "SW11" H 5075 2665 50  0000 C CNN
 F 1 "Switch_tilt" H 5075 2574 50  0000 C CNN
@@
 AR Path="/5D74964C/5E2DF6DD" Ref="SW4"  Part="1"
 AR Path="/5D761BCA/5E2DF6DD" Ref="SW8"  Part="1"
+AR Path="/5EB37636/5E2DF6DD" Ref="SW?"  Part="1"
+AR Path="/5EBCF42E/5E2DF6DD" Ref="SW?"  Part="1"
 F 0 "SW12" H 5075 3115 50  0000 C CNN
 F 1 "Switch_tilt" H 5075 3024 50  0000 C CNN
@@
 AR Path="/5D761BCA/5E6454DE" Ref="R36"  Part="1"
 AR Path="/5D9307E8/5E6454DE" Ref="R45"  Part="1"
+AR Path="/5EB37636/5E6454DE" Ref="R?"  Part="1"
+AR Path="/5EBCF42E/5E6454DE" Ref="R?"  Part="1"
 F 0 "R45" H 3809 2896 50  0000 L CNN
 F 1 "R_Small" H 3809 2805 50  0000 L CNN
@@
 AR Path="/5D761BCA/5D7526E7" Ref="R33"  Part="1"
 AR Path="/5D9307E8/5D7526E7" Ref="R42"  Part="1"
+AR Path="/5EB37636/5D7526E7" Ref="R?"  Part="1"
+AR Path="/5EBCF42E/5D7526E7" Ref="R?"  Part="1"
 F 0 "R42" H 3809 1546 50  0000 L CNN
 F 1 "R_Small" H 3809 1455 50  0000 L CNN
@@
 AR Path="/5D74964C/5E3AEBC9" Ref="#PWR0104"  Part="1"
 AR Path="/5D761BCA/5E3AEBC9" Ref="#PWR0105"  Part="1"
+AR Path="/5EB37636/5E3AEBC9" Ref="#PWR?"  Part="1"
+AR Path="/5EBCF42E/5E3AEBC9" Ref="#PWR?"  Part="1"
 F 0 "#PWR0106" H 3550 2750 50  0001 C CNN
 F 1 "GND" H 3555 2827 50  0000 C CNN
@@
 Wire Wire Line
 	4100 1500 4900 1500
+Text HLabel 2450 3700 1    50   Output ~ 0
+DAC_analog_out
 $EndSCHEMATC
