File: pcb/Luciebox/R2-R_ladder_dac_tilt_switches.sch (KiCad schematic (older format))
At the start: 9 parts, among them SW10 Switch_tilt, SW11 Switch_tilt, SW12 Switch_tilt, SW9 Switch_tilt

Commit message: Restore pcb components
Parts:
- R24, R25, R26, R27: symbol Device:R_Small -> Luciebox_components:R_Small-Device
Changed lines of the file:
@@
 $EndDescr
 $Comp
-L Device:R_Small R26
+L Luciebox_components:R_Small-Device R26
 U 1 1 5D7526DB
 P 3750 2400
@@
 $EndComp
 $Comp
-L Device:R_Small R25
+L Luciebox_components:R_Small-Device R25
 U 1 1 5D7526E1
 P 3750 1950
@@
 $EndComp
 $Comp
-L power:GND #PWR021
+L Luciebox_components:GND-power #PWR021
 U 1 1 5E6454E3
 P 3600 3550
@@
 AR Path="/5EB37636/5E6454E3" Ref="#PWR?"  Part="1"
 AR Path="/5EBCF42E/5E6454E3" Ref="#PWR?"  Part="1"
+AR Path="/5E6454E3" Ref="#PWR027"  Part="1"
 F 0 "#PWR027" H 3600 3300 50  0001 C CNN
 F 1 "GND" H 3605 3377 50  0000 C CNN
@@
 Connection ~ 5750 1500
 $Comp
-L Device:R_Small R27
+L Luciebox_components:R_Small-Device R27
 U 1 1 5E6454DE
 P 3750 2850
@@
 $EndComp
 $Comp
-L Device:R_Small R24
+L Luciebox_components:R_Small-Device R24
 U 1 1 5D7526E7
 P 3750 1500
@@
 Connection ~ 3550 2400
 $Comp
-L power:GND #PWR0106
+L Luciebox_components:GND-power #PWR0106
 U 1 1 5E3AEBC9
 P 3550 3000
@@
 AR Path="/5EB37636/5E3AEBC9" Ref="#PWR?"  Part="1"
 AR Path="/5EBCF42E/5E3AEBC9" Ref="#PWR?"  Part="1"
+AR Path="/5E3AEBC9" Ref="#PWR0106"  Part="1"
 F 0 "#PWR0106" H 3550 2750 50  0001 C CNN
 F 1 "GND" H 3555 2827 50  0000 C CNN
