File: pcb/Luciebox/button_pcb_4x_laz16-11_.kicad_pcb (KiCad board)
At the start: 2 copper layers, 100 x 100 mm, 14 parts, among them T5 terminal_8x1, T6 terminal_8x1, T7 terminal_8x1

Commit message: pcb work on button pcb
Parts:
- removed ?: , artwork:virus_corona
- removed G***: LOGO, artwork:virus_corona3
- removed R29, R30, R31, R32, R33, R34, R35, R36: R_Small, Luciebox:1206_0805
- removed R37: DAC_R-2R, Luciebox:SIP-10
- removed T7: terminal_8x1, Luciebox:Terminal_8x1_100mil
- added H1: MountingHole, Luciebox:MountingHole_4.3mm_M4, F.Cu at (64.0, 80.0)
- added H10: MountingHole, Luciebox:MountingHole_4.3mm_M4, F.Cu at (34.8, -11.7)
- added H11: MountingHole, Luciebox:MountingHole_4.3mm_M4, F.Cu at (44.9, -21.8)
- added H12: MountingHole, Luciebox:MountingHole_4.3mm_M4, F.Cu at (55.1, -32.0)
- added H2: MountingHole, Luciebox:MountingHole_4.3mm_M4, F.Cu at (20.0, 80.0)
- added H3: MountingHole, Luciebox:MountingHole_4.3mm_M4, F.Cu at (42.0, 95.6)
- added H4: MountingHole, Luciebox:MountingHole_4.3mm_M4, F.Cu at (14.5, -11.7)
- added H5: MountingHole, Luciebox:MountingHole_4.3mm_M4, F.Cu at (24.6, -21.8)
- added H6: MountingHole, Luciebox:MountingHole_4.3mm_M4, F.Cu at (34.8, -32.0)
- added H7: MountingHole, Luciebox:MountingHole_4.3mm_M4, F.Cu at (24.6, -11.7)
- added H8: MountingHole, Luciebox:MountingHole_4.3mm_M4, F.Cu at (34.8, -21.8)
- added H9: MountingHole, Luciebox:MountingHole_4.3mm_M4, F.Cu at (44.9, -32.0)
- added R1: DAC_R-2R, Luciebox:SIP-10, F.Cu at (14.2, 97.6)
- added R10: R_Small, Luciebox:1206_0805, F.Cu at (60.0, 92.8)
- added R11: R_Small, Luciebox:1206_0805, F.Cu at (60.2, 88.7)
- added R12: R_Small, Luciebox:1206_0805, F.Cu at (63.5, 92.8)
- added R13: R_Small, Luciebox:1206_0805, F.Cu at (65.8, 88.7)
- added R14: R_Small, Luciebox:1206_0805, F.Cu at (68.0, 92.8)
- added R15: R_Small, Luciebox:1206_0805, F.Cu at (71.4, 88.7)
- added R16: R_Small, Luciebox:1206_0805, F.Cu at (71.0, 92.8)
- added R17: R_Small, Luciebox:1206_0805, F.Cu at (77.0, 88.7)
- added R18: R_Small, Luciebox:1206_0805, F.Cu at (79.8, 92.8)
- added R19: DAC_R-2R, Luciebox:SIP-10, F.Cu at (47.5, 43.7)
- added R2: R_Small, Luciebox:1206_0805, F.Cu at (25.4, 92.6)
- added R3: R_Small, Luciebox:1206_0805, F.Cu at (27.2, 88.5)
- added R4: R_Small, Luciebox:1206_0805, F.Cu at (34.8, 90.3)
- added R5: R_Small, Luciebox:1206_0805, F.Cu at (38.9, 88.3)
- added R6: R_Small, Luciebox:1206_0805, F.Cu at (48.0, 92.8)
- added R7: R_Small, Luciebox:1206_0805, F.Cu at (48.2, 88.8)
- added R8: R_Small, Luciebox:1206_0805, F.Cu at (57.0, 92.8)
- added R9: R_Small, Luciebox:1206_0805, F.Cu at (54.4, 88.7)
- added S1: button_laz16-11, Luciebox:button_LAZ16-11, F.Cu at (8.99, 85.7)
- added S2: button_laz16-11, Luciebox:button_LAZ16-11, F.Cu at (31.0, 85.7)
- added S3: button_laz16-11, Luciebox:button_LAZ16-11, F.Cu at (53.0, 85.7)
- added S4: button_laz16-11, Luciebox:button_LAZ16-11, F.Cu at (75.0, 85.7)
- added S5: button_laz16-11, Luciebox:button_LAZ16-11, F.Cu at (11.4, 52.1)
- added S6: button_laz16-11, Luciebox:button_LAZ16-11, F.Cu at (36.1, 52.3)
- added S7: button_laz16-11, Luciebox:button_LAZ16-11, F.Cu at (61.7, 52.3)
- added S8: button_laz16-11, Luciebox:button_LAZ16-11, F.Cu at (85.6, 50.3)
- added T1: terminal_8x1, Luciebox:Terminal_8x1_100mil, F.Cu at (40.4, 77.6)
- added T2: terminal_8x1, Luciebox:Terminal_8x1_100mil, F.Cu at (11.4, 90.0)
- added T3: terminal_8x1, Luciebox:Terminal_8x1_100mil, F.Cu at (75.9, 41.7)
- added T4: terminal_8x1, Luciebox:Terminal_8x1_100mil, F.Cu at (47.7, 40.4)
- added U1: 4digit_7segments_common_anode_CA56-12SRWA, Display_7Segment:CA56-12SRWA, F.Cu at (161.4, -3.53)
- added connect_for_vcc_as_common_anode1: R_Small, Luciebox:1206_0805, F.Cu at (9.40, 76.8)
- added connect_for_vcc_as_common_anode2: R_Small, Luciebox:1206_0805, F.Cu at (72.1, 44.7)
- moved T5 150.8 mm to (170.9, 2.39), turned to 0 degrees
- moved T6 146.6 mm to (170.9, 6.51), turned to 0 degrees
Connections:
- T5 pad 1: VCC_minimalCurrent -> Net-(T5-Pad1)
- T5 pad 2: VCC_minimalCurrent -> Net-(T5-Pad2)
- T5 pad 3: VCC_minimalCurrent -> Net-(T5-Pad3)
- T5 pad 4: VCC_minimalCurrent -> Net-(T5-Pad4)
- T5 pad 5: VCC_minimalCurrent -> Net-(T5-Pad5)
- T5 pad 6: VCC_minimalCurrent -> Net-(T5-Pad6)
- T5 pad 7: VCC_minimalCurrent -> Net-(T5-Pad7)
- T5 pad 8: VCC_minimalCurrent -> Net-(T5-Pad8)
- T6 pad 1: GND -> Net-(T6-Pad1)
- T6 pad 2: GND -> Net-(T6-Pad2)
- T6 pad 3: GND -> Net-(T6-Pad3)
- T6 pad 4: GND -> Net-(T6-Pad4)
- T6 pad 5: GND -> Net-(T6-Pad5)
- T6 pad 6: GND -> Net-(T6-Pad6)
- T6 pad 7: GND -> Net-(T6-Pad7)
- T6 pad 8: GND -> Net-(T6-Pad8)
Routing:
- net /ANALOG_1: track 0.00 -> 117.3 mm, vias 0 -> 1
- net VCC: track 0.00 -> 111.7 mm, vias 0 -> 2
- net GND: track 30.0 -> 139.0 mm, vias 0 -> 1
- net Net-(S1-Pad4): track 0.00 -> 87.3 mm
- net Net-(R1-Pad3): track 0.00 -> 85.0 mm, vias 0 -> 1
- net Net-(R1-Pad5): track 0.00 -> 84.4 mm, vias 0 -> 2
- net Net-(R1-Pad2): track 0.00 -> 80.8 mm
- net Net-(R1-Pad4): track 0.00 -> 78.4 mm, vias 0 -> 1
- net Net-(R1-Pad7): track 0.00 -> 68.0 mm, vias 0 -> 1
- net Net-(R1-Pad6): track 0.00 -> 65.3 mm, vias 0 -> 1
- net Net-(R1-Pad8): track 0.00 -> 58.6 mm, vias 0 -> 1
- net Net-(S4-Pad5): track 0.00 -> 55.8 mm
- net VCC_minimalCurrent: track 51.8 -> 0.00 mm
- net Net-(S1-Pad5): track 0.00 -> 47.0 mm
- net Net-(R1-Pad9): track 0.00 -> 44.6 mm, vias 0 -> 1
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- removed copper zone on B.Cu, net GND
- removed copper zone on F.Cu, net GND
Other:
- board size 100 x 100 mm -> 100.1 x 99.8 mm
- board text removed: "DAC_A2"
- board text removed: "GND (OFF) NC"
- board text removed: "SWITCH"
- board text removed: "VCC (ON) NO"
