File: pcb/Luciebox/button_pcb_4x_laz16-11_.kicad_pcb (KiCad board)
At the start: 2 copper layers, 100 x 100 mm, 57 parts, among them T1 terminal_8x1, T2 terminal_8x1, T3 terminal_8x1, T4 terminal_8x1, T5 terminal_8x1, T6 terminal_8x1, U1 4digit_7segments_common_anode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

Commit message: before finishing v3
Parts:
- removed the REF** at (78.6, -115.3)
- added H16: MountingHole, Luciebox:MountingHole_4.3mm_M4, F.Cu at (4.50, -34.5)
- added H17: MountingHole, Luciebox:MountingHole_4.3mm_M4, F.Cu at (95.5, -34.5)
Other:
- outline, holes or cut-outs redrawn
Changed lines of the file:
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@@
   (general
     (thickness 1.6)
-    (drawings 64)
+    (drawings 94)
     (tracks 757)
     (zones 0)
-    (modules 57)
+    (modules 58)
     (nets 46)
   )
@@
       (drillshape 0)
       (scaleselection 1)
-      (outputdirectory "Gerber/"))
+      (outputdirectory "Gerber_button_board_v1.0/"))
   )
   (net 0 "")
@@
     (add_net VCC)
   )
+  (module Luciebox:MountingHole_4.3mm_M4 (layer F.Cu)
+    (at 95.5 -34.5)
+    (descr "Mounting Hole 4.3mm, no annular, M4")
+    (tags "mounting hole 4.3mm no annular m4")
+    (attr virtual)
+    (fp_text reference H17 (at 0 -5.3) (layer F.SilkS)
+      (effects (font (size 1 1) (thickness 0.15)))
+    )
+    (fp_text value MountingHole (at 0 5.3) (layer F.Fab)
+      (effects (font (size 1 1) (thickness 0.15)))
+    )
+    (fp_circle (center 0 0) (end 4.55 0) (layer F.CrtYd) (width 0.05))
+    (fp_circle (center 0 0) (end 4.3 0) (layer Cmts.User) (width 0.15))
+    (fp_text user %R (at 0.3 0) (layer F.Fab)
+      (effects (font (size 1 1) (thickness 0.15)))
+    )
+    (pad "" np_thru_hole circle (at 0 0) (size 4.3 4.3) (drill 4.3) (layers *.Cu *.Mask)
+      (clearance 2))
+  )
+  (module Luciebox:MountingHole_4.3mm_M4 (layer F.Cu)
+    (at 4.5 -34.5)
+    (descr "Mounting Hole 4.3mm, no annular, M4")
+    (tags "mounting hole 4.3mm no annular m4")
+    (attr virtual)
+    (fp_text reference H16 (at 0 -5.3) (layer F.SilkS)
+      (effects (font (size 1 1) (thickness 0.15)))
+    )
+    (fp_text value MountingHole (at 0 5.3) (layer F.Fab)
+      (effects (font (size 1 1) (thickness 0.15)))
+    )
+    (fp_circle (center 0 0) (end 4.55 0) (layer F.CrtYd) (width 0.05))
+    (fp_circle (center 0 0) (end 4.3 0) (layer Cmts.User) (width 0.15))
+    (fp_text user %R (at 0.3 0) (layer F.Fab)
+      (effects (font (size 1 1) (thickness 0.15)))
+    )
+    (pad "" np_thru_hole circle (at 0 0) (size 4.3 4.3) (drill 4.3) (layers *.Cu *.Mask)
+      (clearance 2))
+  )
   (module MountingHole:MountingHole_6.4mm_M6 (layer F.Cu)
     (at 93.24 -72.06)
@@
     )
     (pad 1 np_thru_hole circle (at 0 0) (size 3.2 3.2) (drill 3.2) (layers *.Cu *.Mask))
-  )
-  (module MountingHole:MountingHole_4.3mm_M4 (layer F.Cu)
-    (at 78.64 -115.26)
-    (descr "Mounting Hole 4.3mm, no annular, M4")
-    (tags "mounting hole 4.3mm no annular m4")
-    (attr virtual)
-    (fp_text reference REF** (at 0 -5.3) (layer F.SilkS)
-      (effects (font (size 1 1) (thickness 0.15)))
-    )
-    (fp_text value MountingHole_4.3mm_M4 (at 0 5.3) (layer F.Fab)
-      (effects (font (size 1 1) (thickness 0.15)))
-    )
-    (fp_circle (center 0 0) (end 4.55 0) (layer F.CrtYd) (width 0.05))
-    (fp_circle (center 0 0) (end 4.3 0) (layer Cmts.User) (width 0.15))
-    (fp_text user %R (at 0.3 0) (layer F.Fab)
-      (effects (font (size 1 1) (thickness 0.15)))
-    )
-    (pad 1 np_thru_hole circle (at 0 0) (size 4.3 4.3) (drill 4.3) (layers *.Cu *.Mask))
   )
   (module Luciebox:MountingHole_4.3mm_M4 (layer F.Cu)
@@
       ))
   )
-  (gr_text M8 (at 87.54 -62.76) (layer F.SilkS)
+  (gr_line (start 95.64 -27.96) (end 96.14 -27.96) (layer Edge.Cuts) (width 0.1))
+  (gr_line (start 96.14 -55.96) (end 96.14 -40.96) (layer Edge.Cuts) (width 0.1))
+  (gr_line (start 96.14 -40.96) (end 95.64 -40.96) (layer Edge.Cuts) (width 0.1))
+  (gr_line (start 96.14 -11.46) (end 95.64 -11.46) (layer Edge.Cuts) (width 0.1))
+  (gr_line (start 95.64 -40.96) (end 95.64 -55.96) (layer Edge.Cuts) (width 0.1))
+  (gr_line (start 96.14 -27.96) (end 96.14 -11.46) (layer Edge.Cuts) (width 0.1))
+  (gr_line (start 95.64 -11.46) (end 95.64 -27.96) (layer Edge.Cuts) (width 0.1))
+  (gr_line (start 95.64 -55.96) (end 96.14 -55.96) (layer Edge.Cuts) (width 0.1))
+  (gr_line (start 4.14 -27.96) (end 4.14 -11.46) (layer Edge.Cuts) (width 0.1))
+  (gr_line (start 3.64 -27.96) (end 4.14 -27.96) (layer Edge.Cuts) (width 0.1))
+  (gr_line (start 3.64 -11.46) (end 3.64 -27.96) (layer Edge.Cuts) (width 0.1))
+  (gr_line (start 4.14 -11.46) (end 3.64 -11.46) (layer Edge.Cuts) (width 0.1))
+  (gr_line (start 4.14 -55.96) (end 4.14 -40.96) (layer Edge.Cuts) (width 0.1))
+  (gr_line (start 3.64 -55.96) (end 4.14 -55.96) (layer Edge.Cuts) (width 0.1))
+  (gr_line (start 3.64 -40.96) (end 3.64 -55.96) (layer Edge.Cuts) (width 0.1))
+  (gr_line (start 4.14 -40.96) (end 3.64 -40.96) (layer Edge.Cuts) (width 0.1))
+  (gr_line (start 0.64 -16.96) (end 0.64 -14.46) (layer F.SilkS) (width 0.15))
+  (gr_line (start 1.14 -16.96) (end 0.64 -16.96) (layer F.SilkS) (width 0.15))
+  (gr_line (start 1.14 -15.96) (end 1.14 -16.96) (layer F.SilkS) (width 0.15))
+  (gr_line (start 1.64 -15.96) (end 1.14 -15.96) (layer F.SilkS) (width 0.15))
+  (gr_line (start 1.64 -16.96) (end 1.64 -15.96) (layer F.SilkS) (width 0.15))
+  (gr_line (start 2.14 -16.96) (end 1.64 -16.96) (layer F.SilkS) (width 0.15))
+  (gr_line (start 2.14 -16.46) (end 2.14 -16.96) (layer F.SilkS) (width 0.15))
+  (gr_line (start 2.64 -16.46) (end 2.14 -16.46) (layer F.SilkS) (width 0.15))
+  (gr_line (start 2.64 -16.96) (end 2.64 -16.46) (layer F.SilkS) (width 0.15))
+  (gr_line (start 3.14 -16.96) (end 2.64 -16.96) (layer F.SilkS) (width 0.15))
+  (gr_line (start 3.14 -15.96) (end 3.14 -16.96) (layer F.SilkS) (width 0.15))
+  (gr_line (start 2.14 -15.96) (end 3.14 -15.96) (layer F.SilkS) (width 0.15))
+  (gr_line (start 2.14 -14.96) (end 2.14 -15.96) (layer F.SilkS) (width 0.15))
+  (gr_line (start 2.64 -14.96) (end 2.14 -14.96) (layer F.SilkS) (width 0.15))
+  (gr_line (start 2.64 -15.46) (end 2.64 -14.96) (layer F.SilkS) (width 0.15))
+  (gr_line (start 3.14 -15.46) (end 2.64 -15.46) (layer F.SilkS) (width 0.15))
+  (gr_line (start 3.14 -14.46) (end 3.14 -15.46) (layer F.SilkS) (width 0.15))
+  (gr_line (start 1.64 -14.46) (end 3.14 -14.46) (layer F.SilkS) (width 0.15))
+  (gr_line (start 1.64 -15.46) (end 1.64 -14.46) (layer F.SilkS) (width 0.15))
+  (gr_line (start 1.14 -15.46) (end 1.64 -15.46) (layer F.SilkS) (width 0.15))
+  (gr_line (start 1.14 -14.46) (end 1.14 -15.46) (layer F.SilkS) (width 0.15))
+  (gr_line (start 0.64 -14.46) (end 1.14 -14.46) (layer F.SilkS) (width 0.15))
+  (gr_text M8 (at 87.44 -65.26) (layer F.SilkS)
     (effects (font (size 1 1) (thickness 0.15)))
   )
@@
     (effects (font (size 5 5) (thickness 1)))
   )
-  (gr_line (start 95.64 -55.96) (end 95.64 -11.96) (layer Edge.Cuts) (width 0.1))
-  (gr_line (start 94.64 -55.96) (end 95.64 -55.96) (layer Edge.Cuts) (width 0.1))
-  (gr_line (start 94.64 -11.96) (end 94.64 -55.96) (layer Edge.Cuts) (width 0.1))
-  (gr_line (start 95.64 -11.96) (end 94.64 -11.96) (layer Edge.Cuts) (width 0.1))
-  (gr_line (start 5.64 -53.96) (end 5.64 -11.96) (layer Edge.Cuts) (width 0.1))
-  (gr_line (start 4.64 -53.96) (end 5.64 -53.96) (layer Edge.Cuts) (width 0.1))
-  (gr_line (start 4.64 -11.96) (end 4.64 -53.96) (layer Edge.Cuts) (width 0.1))
-  (gr_line (start 5.64 -11.96) (end 4.64 -11.96) (layer Edge.Cuts) (width 0.1))
   (gr_line (start 10.64 -33.96) (end 10.14 -33.46) (layer B.SilkS) (width 0.15))
   (gr_line (start 9.64 -33.96) (end 10.14 -33.46) (layer B.SilkS) (width 0.15))
@@
     (effects (font (size 1 1) (thickness 0.2)) (justify mirror))
   )
-  (via (at 92.64 -60.46) (size 8.6) (drill 8.4) (layers F.Cu B.Cu) (net 0))
+  (via (at 91.44 -61.06) (size 8.6) (drill 8.4) (layers F.Cu B.Cu) (net 0))
   (segment (start 34 -45.008) (end 34 -43.5) (width 0.508) (layer F.Cu) (net 1))
   (segment (start 34 -45.798) (end 34 -45.008) (width 0.508) (layer F.Cu) (net 1))
