File: pcb/Luciebox/button_pcb_4x_laz16-11_.kicad_pcb (KiCad board)
At the start: 2 copper layers, 100 x 100 mm, 67 parts, among them T1 terminal_8x1, T2 terminal_8x1, T3 terminal_8x1, T4 terminal_8x1, T5 terminal_8x1, T6 terminal_8x1, U1 4digit_7segments_common_anode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

Commit message: Pcb v4 setup with kicad6. Button board --> before erasing smd components from the board
Other:
- net class Default removed
