File: pcb/Luciebox/Luciebox_v3.sch (KiCad schematic (older format))
At the start: 62 parts, among them J4 Screw_Terminal_01x07, J5 Screw_Terminal_01x07, J7 USB_B_Mini, P1 CONN_01X01, P2 CONN_01X01, P3 CONN_01X01, P4 CONN_01X01, P5 Digital, P6 Power, P7 Digital, P8 Analog, Q2 N-Channel_Mosfet, T1 terminal_3x1, T13 terminal_8x1, T2 terminal_8x1, T3 terminal_8x1, T4 terminal_3x1, T5 terminal_3x1, T6 terminal_3x1, T8 terminal_3x1, T9 terminal_8x1, U1 CA56-12SRWA, U3 ATmega328-PU, U4 8X8PADS, Y1 16MHz

Commit message: pcb work on button pcb
Parts:
- H1, H2, H3, H4, H5, H6, H7, H8: footprint MountingHole:MountingHole_4mm -> Luciebox:MountingHole_4.3mm_M4; symbol Mechanical:MountingHole -> Luciebox_components:MountingHole

Commit message: before finishing v3
Connections:
- net 0(Rx): now also T13.5, T2.5; no longer T13.1, T2.1, T3.1
- net 1(Tx): now also T13.2, T3.6, U1.5 (g)
- net 12(MISO): now also T13.7, T2.7; no longer T13.3, T2.4, T3.4
- net 13(SCK): now also T3.8; no longer T2.3, T3.3
- net 4: now also T13.3, T3.7; no longer T13.8
- net 7: now also T13.8, T2.8; no longer T13.5
- net 8: now also T13.6, T2.6; no longer T13.2
- net A1: now also T2.3; no longer T3.8
- net A2: now also T3.3; no longer T2.8
- net A3: now also T13.1, T3.5; no longer T13.6
- net GND: now also T2.1, T3.1; no longer T2.7, T3.7
- net VCC_minimalCurrent: now also T2.2, T3.2; no longer T2.6, T3.6
- net at R1.1, T9.1, T9.2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: now also T2.4, T3.4; no longer T2.5, T3.5
- removed net 1: T13.7, T2.2, T3.2, U1.5 (g)
Other:
- moved on the sheet: T13, T9
Changed lines of the file:
@@
 F2 "DAC_analog_out" O R 1300 1200 50
 $EndSheet
-Wire Wire Line
-	3950 3300 3700 3300
-Wire Wire Line
-	3950 3400 3500 3400
-Wire Wire Line
-	3950 3500 3750 3500
-Wire Wire Line
-	3950 3700 3550 3700
-Wire Wire Line
-	3950 3800 3600 3800
-Wire Wire Line
-	3950 3900 3650 3900
-Wire Wire Line
-	3950 4000 3450 4000
-Wire Wire Line
-	3950 3600 3800 3600
 Connection ~ 5000 3400
 Wire Wire Line
 	5000 3300 5000 3400
 Wire Wire Line
-	4750 3300 5000 3300
+	4950 3300 5000 3300
 Connection ~ 5000 3500
 Wire Wire Line
 	5000 3400 5000 3500
 Wire Wire Line
-	4750 3400 5000 3400
+	4950 3400 5000 3400
 Connection ~ 5000 3600
 Wire Wire Line
 	5000 3500 5000 3600
 Wire Wire Line
-	4750 3500 5000 3500
+	4950 3500 5000 3500
 Connection ~ 5000 3700
 Wire Wire Line
 	5000 3600 5000 3700
 Wire Wire Line
-	4750 3600 5000 3600
+	4950 3600 5000 3600
 Connection ~ 5000 3800
 Wire Wire Line
-	5000 3700 4750 3700
+	5000 3700 4950 3700
 Wire Wire Line
 	5000 3800 5000 3700
@@
 	5000 3800 5000 3900
 Wire Wire Line
-	4750 3800 5000 3800
-Wire Wire Line
-	4750 3900 5000 3900
-Wire Wire Line
-	4750 4000 5000 4000
+	4950 3800 5000 3800
+Wire Wire Line
+	4950 3900 5000 3900
+Wire Wire Line
+	4950 4000 5000 4000
 Wire Wire Line
 	5000 3900 5000 4000
 Wire Wire Line
-	5000 2300 5000 3300
+	5000 2300 5000 3050
 Connection ~ 5000 3300
 Wire Wire Line
 	5000 2300 6500 2300
-Wire Wire Line
-	3450 1700 3450 1750
-Wire Wire Line
-	3800 1000 3800 3600
-Wire Wire Line
-	3750 1100 3750 3500
-Wire Wire Line
-	3700 1200 3700 3300
-Wire Wire Line
-	3650 1300 3650 3900
-Wire Wire Line
-	3600 1400 3600 2050
-Wire Wire Line
-	3550 1500 3550 1950
-Wire Wire Line
-	3500 1600 3500 1850
-Text Label 2450 3450 0    50   ~ 0
+Text Label 2450 1950 0    50   ~ 0
 A1
-Text Label 2450 2450 0    50   ~ 0
+Text Label 2450 2950 0    50   ~ 0
 A2
-Wire Wire Line
-	2450 1750 3450 1750
-Connection ~ 3450 1750
-Wire Wire Line
-	3450 1750 3450 2750
-Wire Wire Line
-	2450 1850 3500 1850
-Connection ~ 3500 1850
-Wire Wire Line
-	3500 1850 3500 2850
-Wire Wire Line
-	2450 1950 3550 1950
-Connection ~ 3550 1950
-Wire Wire Line
-	3550 1950 3550 2950
-Wire Wire Line
-	2450 2050 3600 2050
-Connection ~ 3600 2050
-Wire Wire Line
-	3600 2050 3600 3050
-Wire Wire Line
-	2450 2750 3450 2750
-Connection ~ 3450 2750
-Wire Wire Line
-	3450 2750 3450 4000
-Wire Wire Line
-	2450 2850 3500 2850
-Connection ~ 3500 2850
-Wire Wire Line
-	3500 2850 3500 3400
-Wire Wire Line
-	2450 2950 3550 2950
-Connection ~ 3550 2950
-Wire Wire Line
-	3550 2950 3550 3700
-Connection ~ 3600 3050
-Wire Wire Line
-	3600 3050 3600 3800
-Wire Wire Line
-	2450 2150 3300 2150
-Wire Wire Line
-	5000 2150 5000 2300
 Connection ~ 5000 2300
-Wire Wire Line
-	2450 3150 3300 3150
-Wire Wire Line
-	3300 3150 3300 2150
-Connection ~ 3300 2150
-Wire Wire Line
-	3300 2150 5000 2150
 $Comp
 L power:GND #PWR0103
 U 1 1 5FFAF02F
-P 2850 2350
-F 0 "#PWR0103" H 2850 2100 50  0001 C CNN
-F 1 "GND" H 2855 2177 50  0000 C CNN
-F 2 "" H 2850 2350 50  0001 C CNN
-F 3 "" H 2850 2350 50  0001 C CNN
-	1    2850 2350
+P 3150 1750
+F 0 "#PWR0103" H 3150 1500 50  0001 C CNN
+F 1 "GND" H 3155 1577 50  0000 C CNN
+F 2 "" H 3150 1750 50  0001 C CNN
+F 3 "" H 3150 1750 50  0001 C CNN
+	1    3150 1750
 	1    0    0    -1
 $EndComp
@@
 L power:GND #PWR0107
 U 1 1 5FFAF53B
-P 2850 3350
-F 0 "#PWR0107" H 2850 3100 50  0001 C CNN
-F 1 "GND" H 2855 3177 50  0000 C CNN
-F 2 "" H 2850 3350 50  0001 C CNN
-F 3 "" H 2850 3350 50  0001 C CNN
-	1    2850 3350
-	1    0    0    -1
-$EndComp
-Wire Wire Line
-	2450 3350 2850 3350
-Wire Wire Line
-	2450 2350 2850 2350
+P 3150 2750
+F 0 "#PWR0107" H 3150 2500 50  0001 C CNN
+F 1 "GND" H 3155 2577 50  0000 C CNN
+F 2 "" H 3150 2750 50  0001 C CNN
+F 3 "" H 3150 2750 50  0001 C CNN
+	1    3150 2750
+	1    0    0    -1
+$EndComp
 $Comp
 L Luciebox_components:VCC_minimalCurrent #PWR0108
 U 1 1 5FFE60B8
-P 2950 3650
-F 0 "#PWR0108" H 2950 3500 50  0001 C CNN
-F 1 "VCC_minimalCurrent" H 2967 3823 50  0000 C CNN
-F 2 "" H 2950 3650 50  0001 C CNN
-F 3 "" H 2950 3650 50  0001 C CNN
-	1    2950 3650
+P 3050 3650
+F 0 "#PWR0108" H 3050 3500 50  0001 C CNN
+F 1 "VCC_minimalCurrent" H 3067 3823 50  0000 C CNN
+F 2 "" H 3050 3650 50  0001 C CNN
+F 3 "" H 3050 3650 50  0001 C CNN
+	1    3050 3650
 	-1   0    0    1
 $EndComp
-Wire Wire Line
-	2450 2250 3050 2250
-Wire Wire Line
-	3050 2250 3050 3250
-Wire Wire Line
-	3050 3250 2950 3250
-Wire Wire Line
-	2950 3650 2950 3250
-Connection ~ 2950 3250
-Wire Wire Line
-	2950 3250 2450 3250
 Text Label 1250 6000 2    50   ~ 0
 2
@@
 3(PWM)
 Text Label 3350 1600 2    50   ~ 0
-1
+1(Tx)
 Text Label 3350 1100 2    50   ~ 0
 A3
-Wire Wire Line
-	2450 3050 3600 3050
 Wire Wire Line
 	2650 4000 2000 4000
@@
 L Luciebox_components:terminal_8x1 T9
 U 1 1 5E968FAE
-P 4700 4000
-F 0 "T9" H 4817 3785 50  0000 C CNN
-F 1 "terminal_8x1" H 4817 3876 50  0000 C CNN
-F 2 "Luciebox:Terminal_8x1_100mil" H 4500 3900 50  0001 C CNN
-F 3 "" H 4650 5100 50  0001 C CNN
-	1    4700 4000
+P 4900 4000
+F 0 "T9" H 5017 3785 50  0000 C CNN
+F 1 "terminal_8x1" H 5017 3876 50  0000 C CNN
+F 2 "Luciebox:Terminal_8x1_100mil" H 4700 3900 50  0001 C CNN
+F 3 "" H 4850 5100 50  0001 C CNN
+	1    4900 4000
 	-1   0    0    -1
 $EndComp
@@
 L Luciebox_components:terminal_8x1 T13
 U 1 1 5E835E31
-P 4000 4000
-F 0 "T13" H 4117 3785 50  0000 C CNN
-F 1 "terminal_8x1" H 4117 3876 50  0000 C CNN
-F 2 "Luciebox:Terminal_8x1_100mil" H 3800 3900 50  0001 C CNN
-F 3 "" H 3950 5100 50  0001 C CNN
-	1    4000 4000
+P 4250 4000
+F 0 "T13" H 4367 3785 50  0000 C CNN
+F 1 "terminal_8x1" H 4367 3876 50  0000 C CNN
+F 2 "Luciebox:Terminal_8x1_100mil" H 4050 3900 50  0001 C CNN
+F 3 "" H 4200 5100 50  0001 C CNN
+	1    4250 4000
 	1    0    0    -1
 $EndComp
@@
 	1    0    0    -1
 $EndComp
+Wire Wire Line
+	3450 1700 3450 2150
+Wire Wire Line
+	3550 1500 3550 3450
+Wire Wire Line
+	3650 1300 3650 2250
+Wire Wire Line
+	3800 1000 3800 2450
+Wire Wire Line
+	5000 2050 5000 2300
+Wire Wire Line
+	2450 2150 3450 2150
+Connection ~ 3450 2150
+Wire Wire Line
+	3450 2150 3450 4000
+Wire Wire Line
+	2450 1750 3150 1750
+Wire Wire Line
+	2450 1850 3050 1850
+Wire Wire Line
+	3050 1850 3050 2850
+Wire Wire Line
+	3650 2250 2450 2250
+Wire Wire Line
+	2450 2350 3600 2350
+Wire Wire Line
+	3600 1400 3600 2350
+Wire Wire Line
+	2450 2450 3800 2450
+Wire Wire Line
+	2450 2750 3150 2750
+Wire Wire Line
+	2450 2850 3050 2850
+Connection ~ 3050 2850
+Wire Wire Line
+	2450 3050 5000 3050
+Connection ~ 5000 3050
+Wire Wire Line
+	5000 3050 5000 3300
+Wire Wire Line
+	2450 2050 5000 2050
+Wire Wire Line
+	3500 1600 3500 3250
+Wire Wire Line
+	2450 3150 3750 3150
+Wire Wire Line
+	3750 1100 3750 3150
+Wire Wire Line
+	3050 2850 3050 3650
+Wire Wire Line
+	2450 3250 3500 3250
+Wire Wire Line
+	2450 3350 3700 3350
+Wire Wire Line
+	2450 3450 3550 3450
+Text Label 4200 4000 2    50   ~ 0
+A3
+Text Label 4200 3900 2    50   ~ 0
+1(Tx)
+Text Label 4200 3800 2    50   ~ 0
+4
+Text Label 4200 3600 2    50   ~ 0
+0(Rx)
+Text Label 4200 3500 2    50   ~ 0
+8
+Text Label 4200 3400 2    50   ~ 0
+12(MISO)
+Text Label 4200 3300 2    50   ~ 0
+7
+Wire Wire Line
+	3700 1200 3700 3350
+Text Label 4200 3700 2    50   ~ 0
+13(SCK)
 $EndSCHEMATC

Commit message: pcb v3 comming along
Parts:
- removed J7: USB_B_Mini, Luciebox:usb_mini_Molex-0548190519, symbol Connector:USB_B_Mini
- added J1: USB_B_Mini, Luciebox:usb_mini_Molex-0548190519, symbol Luciebox_components:USB_B_Mini
- added T10, T7: terminal_3x1, Luciebox:Terminal_3x1_100mil, symbol Luciebox_components:terminal_3x1
Connections:
- net 13(SCK): now also T7.3
- net 7: now also T7.2
- net A3: now also T10.3
- net GND: now also J1.1 (GND), J1.6 (Shield)
- net at R5.1, U1.12 (CA1): now also T7.1
- net at R3.1, U1.8 (CA3): now also T10.2
- net at R4.1, U1.9 (CA2): now also T10.1
- net at D1.2 (A): now also J1.5 (VBUS)
- net at T8.2: now also J1.4 (D-)
- net at T8.3: now also J1.3 (D+)
- net at T8.1: now also J1.2 (ID)
Changed lines of the file:
@@
 	10700 1000 10700 500
-Wire Wire Line
-	6050 1600 7000 1600
 Wire Wire Line
 	7000 1600 7000 2300
@@
 0(Rx)
 Wire Wire Line
-	3350 1000 3800 1000
+	3350 1000 3750 1000
 Connection ~ 3800 1000
 Wire Wire Line
-	3350 1100 3750 1100
+	3350 1100 3650 1100
 Connection ~ 3750 1100
 Wire Wire Line
@@
 $EndComp
 $Comp
-L Connector:USB_B_Mini J7
-U 1 1 5E641E20
-P 4700 5800
-F 0 "J7" H 4470 5697 50  0000 R CNN
-F 1 "USB_B_Mini" H 4470 5788 50  0000 R CNN
-F 2 "Luciebox:usb_mini_Molex-0548190519" H 4850 5750 50  0001 C CNN
-F 3 "~" H 4850 5750 50  0001 C CNN
-	1    4700 5800
-	-1   0    0    1
-$EndComp
-$Comp
 L Device:R_Small R49
 U 1 1 5E1772EF
@@
 Text Label 4200 3700 2    50   ~ 0
 13(SCK)
+$Comp
+L Luciebox_components:terminal_3x1 T10
+U 1 1 606256A8
+P 2600 1200
+F 0 "T10" H 2692 985 50  0000 C CNN
+F 1 "terminal_3x1" H 2692 1076 50  0000 C CNN
+F 2 "Luciebox:Terminal_3x1_100mil" H 2400 1100 50  0001 C CNN
+F 3 "" H 2550 1600 50  0001 C CNN
+	1    2600 1200
+	-1   0    0    1
+$EndComp
+$Comp
+L Luciebox_components:terminal_3x1 T7
+U 1 1 606246AE
+P 2600 750
+F 0 "T7" H 2692 535 50  0000 C CNN
+F 1 "terminal_3x1" H 2692 626 50  0000 C CNN
+F 2 "Luciebox:Terminal_3x1_100mil" H 2400 650 50  0001 C CNN
+F 3 "" H 2550 1150 50  0001 C CNN
+	1    2600 750
+	-1   0    0    1
+$EndComp
+Wire Wire Line
+	7500 600  2850 600
+Wire Wire Line
+	2850 600  2850 750
+Wire Wire Line
+	2850 750  2650 750
+Wire Wire Line
+	7500 600  7500 1400
+Connection ~ 7500 1400
+Wire Wire Line
+	3750 850  2650 850
+Wire Wire Line
+	3550 1500 3550 950
+Wire Wire Line
+	3550 950  2650 950
+Wire Wire Line
+	7250 1500 7250 650
+Wire Wire Line
+	7250 650  2900 650
+Wire Wire Line
+	2900 650  2900 1200
+Wire Wire Line
+	2900 1200 2650 1200
+Connection ~ 7250 1500
+Wire Wire Line
+	6050 1600 7000 1600
+Wire Wire Line
+	7000 1600 7000 700
+Wire Wire Line
+	7000 700  2950 700
+Wire Wire Line
+	2950 700  2950 1300
+Wire Wire Line
+	2950 1300 2650 1300
+Connection ~ 7000 1600
+Wire Wire Line
+	3750 850  3750 1000
+Connection ~ 3750 1000
+Wire Wire Line
+	3750 1000 3800 1000
+Wire Wire Line
+	3650 1100 3650 750
+Wire Wire Line
+	3650 750  3000 750
+Wire Wire Line
+	3000 750  3000 1400
+Wire Wire Line
+	3000 1400 2650 1400
+Connection ~ 3650 1100
+Wire Wire Line
+	3650 1100 3750 1100
+$Comp
+L Luciebox_components:USB_B_Mini J1
+U 1 1 608A892E
+P 4700 5800
+F 0 "J1" H 4470 5697 50  0000 R CNN
+F 1 "USB_B_Mini" H 4470 5788 50  0000 R CNN
+F 2 "Luciebox:usb_mini_Molex-0548190519" H 4850 5750 50  0001 C CNN
+F 3 "~" H 4850 5750 50  0001 C CNN
+	1    4700 5800
+	-1   0    0    1
+$EndComp
 $EndSCHEMATC

Commit message: published and ordered v3 luciebox v1 buttonboard. Gerbers included
Parts:
- removed J4, J5: Screw_Terminal_01x07, Luciebox:Terminal_7x1_100mil, symbol Connector:Screw_Terminal_01x07
- added R_0_if_no_touch1, R_0_if_no_usb_switch1: 0, Luciebox:1206_0805, symbol Device:R_Small
- added T12, T13: terminal_8x1, Luciebox:Terminal_8x1_100mil, symbol Luciebox_components:terminal_8x1
- added TP1: TestPoint_Probe, symbol Connector:TestPoint_Probe
- R9: renamed from R47; value 100K -> 10K
- renumbered H4 to H1, H1 to H2, H2 to H3, H3 to H4, P6 to P1, P8 to P2, P5 to P3, P7 to P4, P1 to P5, P2 to P6, P3 to P7, P4 to P8, Q2 to Q1, R7 to R1, R48 to R10, R15 to R11, R16 to R12, R17 to R13, R18 to R14, R1 to R15, R2 to R16, R3 to R17, R4 to R18, R5 to R19, R8 to R2, R6 to R20, R9 to R3, R10 to R4, R11 to R5, R12 to R6, R13 to R7, R14 to R8, R19 to R_reset_pullup1, R49 to R_vcc_protected1, S2 to S1, S1 to S2, T13 to T10, T9 to T11, T5 to T2, T4 to T3, T6 to T4, T2 to T5, T3 to T6, T10 to T8, T8 to T9, U4 to U2
Connections:
- wire segments 339 -> 354
Other:
- note added: "GND-EXTERNAL"
- note added: "GND-SWITCHED"
- note added: "SWITCH_BATTERY_POWER"
- note added: "SWITCH_USB_POWER"
- note removed: "MASTER-ON"
- note removed: "TOUCH-ON"
- moved on the sheet: Q1, R10, R9

Commit message: Restore pcb components
Parts:
- BZ1: symbol Device:Buzzer -> Luciebox_components:Buzzer-Device
- C1, C2, C3: symbol Device:C_Small -> Luciebox_components:C_Small-Device
- P1, P4: symbol Connector_Generic:Conn_01x08 -> Luciebox_components:Conn_01x08-Connector_Generic
- P2: symbol Connector_Generic:Conn_01x06 -> Luciebox_components:Conn_01x06-Connector_Generic
- P3: symbol Connector_Generic:Conn_01x10 -> Luciebox_components:Conn_01x10-Connector_Generic
- P5, P6, P7, P8: symbol Connector_Generic:Conn_01x01 -> Luciebox_components:Conn_01x01-Connector_Generic
- R1, R10, R11, R12, R13, R14, R15, R16, R17, R18, R19, R2, R20, R3, R4, R5, R6, R7, R8, R9, R_0_if_no_touch1, R_0_if_no_usb_switch1, R_reset_pullup1, R_vcc_protected1: symbol Device:R_Small -> Luciebox_components:R_Small-Device
- Y1: symbol Device:Crystal -> Luciebox_components:Crystal-Device
Connections:
- net labels added: GND-power
Changed lines of the file:
@@
 Reset
 $Comp
-L power:+3.3V #PWR020
+L Luciebox_components:+3.3V-power #PWR020
 U 1 1 56D70538
 P 9150 1450
@@
 $EndComp
 $Comp
-L power:VCC #PWR019
+L Luciebox_components:VCC-power #PWR019
 U 1 1 56D707BB
 P 9050 1350
@@
 $EndComp
 $Comp
-L power:GND #PWR021
+L Luciebox_components:GND-power #PWR021
 U 1 1 56D70CC2
 P 9300 3150
@@
 $EndComp
 $Comp
-L power:GND #PWR023
+L Luciebox_components:GND-power #PWR023
 U 1 1 56D70CFF
 P 10300 3150
@@
 	850  4900 800  4900
 $Comp
-L power:GND #PWR01
+L Luciebox_components:GND-power #PWR01
 U 1 1 5D7F94C7
 P 700 4900
@@
 A0
 $Comp
-L power:GND #PWR03
+L Luciebox_components:GND-power #PWR03
 U 1 1 5D90E4DE
 P 1100 6200
@@
 	1500 6850 2000 6850
 $Comp
-L power:GND #PWR05
+L Luciebox_components:GND-power #PWR05
 U 1 1 5D974320
 P 2000 6850
@@
 A5(SCL)
 $Comp
-L power:GND #PWR017
+L Luciebox_components:GND-power #PWR017
 U 1 1 5D988298
 P 7900 6450
@@
 7
 $Comp
-L power:VCC #PWR016
+L Luciebox_components:VCC-power #PWR016
 U 1 1 5D991DF2
 P 7900 3450
@@
 $EndComp
 $Comp
-L power:VCC #PWR018
+L Luciebox_components:VCC-power #PWR018
 U 1 1 5D992AD7
 P 8000 3450
@@
 $EndComp
 $Comp
-L power:VCC #PWR015
+L Luciebox_components:VCC-power #PWR015
 U 1 1 5D993297
 P 7300 3750
@@
 	10500 4700 10350 4700
 $Comp
-L power:GND #PWR024
+L Luciebox_components:GND-power #PWR024
 U 1 1 5DA1D313
 P 10700 4500
 F 0 "#PWR024" H 10700 4250 50  0001 C CNN
-F 1 "GND" H 10700 4350 50  0000 C CNN
+F 1 "GND-power" H 10700 4350 50  0000 C CNN
 F 2 "" H 10700 4500 50  0000 C CNN
 F 3 "" H 10700 4500 50  0000 C CNN
@@
 Connection ~ 7900 3450
 $Comp
-L power:GND #PWR014
+L Luciebox_components:GND-power #PWR014
 U 1 1 5DA38582
 P 6700 3400
@@
 	9400 5250 9250 5250
 $Comp
-L power:VCC #PWR022
+L Luciebox_components:VCC-power #PWR022
 U 1 1 5DA5FE62
 P 9900 5250
@@
 A4(SDA)
 $Comp
-L power:GND #PWR09
+L Luciebox_components:GND-power #PWR09
 U 1 1 5D70EC69
 P 3950 6400
@@
 	5700 7250 5150 7250
 $Comp
-L power:VCC #PWR011
+L Luciebox_components:VCC-power #PWR011
 U 1 1 5D7FF3DB
 P 5000 7150
@@
 	6300 4500 6300 4400
 $Comp
-L power:GND #PWR013
+L Luciebox_components:GND-power #PWR013
 U 1 1 5DCBF971
 P 6450 4700
@@
 $EndComp
 $Comp
-L power:VCC #PWR012
+L Luciebox_components:VCC-power #PWR012
 U 1 1 5DCC8327
 P 5400 4000
@@
 Connection ~ 6450 4700
 $Comp
-L power:VCC #PWR04
+L Luciebox_components:VCC-power #PWR04
 U 1 1 5E19FB8B
 P 1550 2400
@@
 Connection ~ 5000 2300
 $Comp
-L power:GND #PWR07
+L Luciebox_components:GND-power #PWR07
 U 1 1 5FFAF02F
 P 3150 1750
@@
 $EndComp
 $Comp
-L power:GND #PWR08
+L Luciebox_components:GND-power #PWR08
 U 1 1 5FFAF53B
 P 3150 2750
@@
 $EndComp
 $Comp
-L Device:R_Small R_vcc_protected1
+L Luciebox_components:R_Small-Device R_vcc_protected1
 U 1 1 5E1772EF
 P 1450 2400
@@
 $EndComp
 $Comp
-L Device:R_Small R10
+L Luciebox_components:R_Small-Device R10
 U 1 1 5D6C3ACD
 P 3100 7000
@@
 $EndComp
 $Comp
-L Device:R_Small R9
+L Luciebox_components:R_Small-Device R9
 U 1 1 5D6C3437
 P 3100 6600
@@
 $EndComp
 $Comp
-L Device:R_Small R_reset_pullup1
+L Luciebox_components:R_Small-Device R_reset_pullup1
 U 1 1 5DA45BE6
 P 9500 5250
@@
 $EndComp
 $Comp
-L Device:C_Small C1
+L Luciebox_components:C_Small-Device C1
 U 1 1 5DA2A1AC
 P 6950 3400
@@
 $EndComp
 $Comp
-L Device:C_Small C3
+L Luciebox_components:C_Small-Device C3
 U 1 1 5D9EAF46
 P 10250 4700
@@
 $EndComp
 $Comp
-L Device:C_Small C2
+L Luciebox_components:C_Small-Device C2
 U 1 1 5D9EA27E
 P 10250 4350
@@
 $EndComp
 $Comp
-L Device:R_Small R20
+L Luciebox_components:R_Small-Device R20
 U 1 1 5D9BA081
 P 9300 4450
@@
 $EndComp
 $Comp
-L Device:Crystal Y1
+L Luciebox_components:Crystal-Device Y1
 U 1 1 5D9962E4
 P 9750 4500
@@
 $EndComp
 $Comp
-L Device:Buzzer BZ1
+L Luciebox_components:Buzzer-Device BZ1
 U 1 1 5D93C6F4
 P 1400 6750
@@
 $EndComp
 $Comp
-L Device:R_Small R14
+L Luciebox_components:R_Small-Device R14
 U 1 1 5D7D8CC8
 P 4250 4900
@@
 $EndComp
 $Comp
-L Device:R_Small R13
+L Luciebox_components:R_Small-Device R13
 U 1 1 5D7D8CBE
 P 3950 4900
@@
 $EndComp
 $Comp
-L Device:R_Small R12
+L Luciebox_components:R_Small-Device R12
 U 1 1 5D7D8CB3
 P 3650 4900
@@
 $EndComp
 $Comp
-L Device:R_Small R11
+L Luciebox_components:R_Small-Device R11
 U 1 1 5D7D8CA9
 P 3350 4900
@@
 $EndComp
 $Comp
-L Device:R_Small R8
+L Luciebox_components:R_Small-Device R8
 U 1 1 5D7CF8D8
 P 3050 4900
@@
 $EndComp
 $Comp
-L Device:R_Small R7
+L Luciebox_components:R_Small-Device R7
 U 1 1 5D7CF8CE
 P 2750 4900
@@
 $EndComp
 $Comp
-L Device:R_Small R6
+L Luciebox_components:R_Small-Device R6
 U 1 1 5D7CF8C3
 P 2450 4900
@@
 $EndComp
 $Comp
-L Device:R_Small R5
+L Luciebox_components:R_Small-Device R5
 U 1 1 5D7CF8B9
 P 2150 4900
@@
 $EndComp
 $Comp
-L Device:R_Small R4
+L Luciebox_components:R_Small-Device R4
 U 1 1 5D7B59FE
 P 1850 4900
@@
 $EndComp
 $Comp
-L Device:R_Small R3
+L Luciebox_components:R_Small-Device R3
 U 1 1 5D7B59F4
 P 1550 4900
@@
 $EndComp
 $Comp
-L Device:R_Small R2
+L Luciebox_components:R_Small-Device R2
 U 1 1 5D79CF90
 P 1250 4900
@@
 $EndComp
 $Comp
-L Device:R_Small R1
+L Luciebox_components:R_Small-Device R1
 U 1 1 5D798401
 P 950 4900
@@
 $EndComp
 $Comp
-L Device:R_Small R15
+L Luciebox_components:R_Small-Device R15
 U 1 1 5D4E6F2F
 P 6500 2400
@@
 $EndComp
 $Comp
-L Device:R_Small R16
+L Luciebox_components:R_Small-Device R16
 U 1 1 5D496C09
 P 6750 2400
@@
 $EndComp
 $Comp
-L Device:R_Small R19
+L Luciebox_components:R_Small-Device R19
 U 1 1 5D49796F
 P 7500 2400
@@
 $EndComp
 $Comp
-L Device:R_Small R18
+L Luciebox_components:R_Small-Device R18
 U 1 1 5D497707
 P 7250 2400
@@
 $EndComp
 $Comp
-L Device:R_Small R17
+L Luciebox_components:R_Small-Device R17
 U 1 1 5D49734E
 P 7000 2400
@@
 $EndComp
 $Comp
-L Connector_Generic:Conn_01x10 P3
+L Luciebox_components:Conn_01x10-Connector_Generic P3
 U 1 1 56D721E0
 P 10000 1600
@@
 $EndComp
 $Comp
-L Connector_Generic:Conn_01x08 P4
+L Luciebox_components:Conn_01x08-Connector_Generic P4
 U 1 1 56D7164F
 P 10000 2600
@@
 $EndComp
 $Comp
-L Connector_Generic:Conn_01x01 P8
+L Luciebox_components:Conn_01x01-Connector_Generic P8
 U 1 1 56D712DB
 P 11100 650
@@
 $EndComp
 $Comp
-L Connector_Generic:Conn_01x01 P7
+L Luciebox_components:Conn_01x01-Connector_Generic P7
 U 1 1 56D712A8
 P 11000 650
@@
 $EndComp
 $Comp
-L Connector_Generic:Conn_01x01 P6
+L Luciebox_components:Conn_01x01-Connector_Generic P6
 U 1 1 56D71274
 P 10900 650
@@
 $EndComp
 $Comp
-L Connector_Generic:Conn_01x01 P5
+L Luciebox_components:Conn_01x01-Connector_Generic P5
 U 1 1 56D71177
 P 10800 650
@@
 $EndComp
 $Comp
-L Connector_Generic:Conn_01x06 P2
+L Luciebox_components:Conn_01x06-Connector_Generic P2
 U 1 1 56D70DD8
 P 9600 2700
@@
 $EndComp
 $Comp
-L Connector_Generic:Conn_01x08 P1
+L Luciebox_components:Conn_01x08-Connector_Generic P1
 U 1 1 56D70129
 P 9600 1900
@@
 	4800 5350 5350 5350
 $Comp
-L Device:R_Small R_0_if_no_touch1
+L Luciebox_components:R_Small-Device R_0_if_no_touch1
 U 1 1 5FE57FC5
 P 5150 6500
@@
 	5100 7150 5700 7150
 $Comp
-L Device:R_Small R_0_if_no_usb_switch1
+L Luciebox_components:R_Small-Device R_0_if_no_usb_switch1
 U 1 1 5FF3108A
 P 5250 7550
