File: pcb/Luciebox_v4 - Copy/Luciebox_buttons.kicad_sch (KiCad schematic)
At the start: 61 parts, among them T14 terminal_8x1, T15 terminal_8x1, T16 terminal_8x1, T17 terminal_8x1, T18 terminal_8x1, T19 terminal_8x1, U4 4digit_7segments_common_anode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

Commit message: V4 main pcb ready for layouting
Parts:
- renumbered D4 to D?, D6 to D?, D5 to D?, D9 to D?, D2 to D?, D8 to D?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
