File: pcb/Luciebox_v4/main_pcb/Luciebox_v4.kicad_pcb (KiCad board)
At the start: 2 copper layers, 78 x 92 mm, 64 parts, among them J1 USB_B_Mini, J2 USB_B_Mini, Q1 P-Channel MOSFET, Q2 NPN transistor, T1 terminal_8x1, T2 terminal_3x1, T4 terminal_8x1, T5 terminal_3x1, T6 terminal_8x1, T7 terminal_8x1, T8 terminal_8x1, U1 CA56-12SRWA, U2 8X8PADS, U3 ATmega328-PU, Y1 16MHz

Commit message: Moved boards connector. Main board ready for traces.
Parts:
- moved T5 9.80 mm to (10.2, 72.9), turned to 90 degrees
- moved U2 3.36 mm to (22.7, 77.2)
- moved T1 2.00 mm to (39.4, 88.6)
- moved T4 2.00 mm to (59.7, 88.6)
- moved T6 2.00 mm to (19.1, 88.6)
- moved J1 1.78 mm to (0.10, 73.6)
- moved S1 1.02 mm to (12.7, 49.6)
Connections:
- U2 pad 25: unconnected-(U2-Pad25) -> Net-(U2-Pad25)
- U2 pad 26: unconnected-(U2-Pad26) -> Net-(U2-Pad25)
- U2 pad 27: unconnected-(U2-Pad27) -> Net-(U2-Pad27)
- U2 pad 28: unconnected-(U2-Pad28) -> Net-(U2-Pad27)
- U2 pad 29: unconnected-(U2-Pad29) -> Net-(U2-Pad29)
- U2 pad 30: Net-(U2-Pad30) -> Net-(U2-Pad29)
- U2 pad 31: Net-(U2-Pad30) -> Net-(U2-Pad29)
- U2 pad 32: Net-(U2-Pad30) -> Net-(U2-Pad29)
- U2 pad 33: unconnected-(U2-Pad33) -> Net-(U2-Pad33)
- U2 pad 34: unconnected-(U2-Pad34) -> Net-(U2-Pad33)
- U2 pad 35: unconnected-(U2-Pad35) -> Net-(U2-Pad35)
- U2 pad 36: unconnected-(U2-Pad36) -> Net-(U2-Pad35)
- U2 pad 37: unconnected-(U2-Pad37) -> Net-(U2-Pad37)
- U2 pad 38: Net-(U2-Pad38) -> Net-(U2-Pad37)
- U2 pad 39: Net-(U2-Pad38) -> Net-(U2-Pad37)
- U2 pad 40: Net-(U2-Pad38) -> Net-(U2-Pad37)
- U2 pad 41: unconnected-(U2-Pad41) -> Net-(U2-Pad41)
- U2 pad 42: unconnected-(U2-Pad42) -> Net-(U2-Pad41)
- U2 pad 43: unconnected-(U2-Pad43) -> Net-(U2-Pad43)
- U2 pad 44: unconnected-(U2-Pad44) -> Net-(U2-Pad43)
- U2 pad 45: unconnected-(U2-Pad45) -> Net-(U2-Pad45)
- U2 pad 46: Net-(U2-Pad46) -> Net-(U2-Pad45)
- U2 pad 47: Net-(U2-Pad46) -> Net-(U2-Pad45)
- U2 pad 48: Net-(U2-Pad46) -> Net-(U2-Pad45)
- U2 pad 49: unconnected-(U2-Pad49) -> Net-(U2-Pad49)
- U2 pad 50: unconnected-(U2-Pad50) -> Net-(U2-Pad49)
- U2 pad 51: unconnected-(U2-Pad51) -> Net-(U2-Pad51)
- U2 pad 52: unconnected-(U2-Pad52) -> Net-(U2-Pad51)
- U2 pad 53: unconnected-(U2-Pad53) -> Net-(U2-Pad53)
- U2 pad 54: Net-(U2-Pad54) -> Net-(U2-Pad53)
- U2 pad 55: Net-(U2-Pad54) -> Net-(U2-Pad53)
- U2 pad 56: Net-(U2-Pad54) -> Net-(U2-Pad53)
Routing:
- net GND: track 0.00 -> 17.8 mm
- net VCC: track 0.00 -> 15.3 mm
- net Net-(U2-Pad45): track 0.00 -> 7.64 mm
- net Net-(U2-Pad53): track 0.00 -> 7.64 mm
- net Net-(U2-Pad37): track 0.00 -> 7.64 mm
- net Net-(U2-Pad13): track 0.00 -> 5.11 mm
- net Net-(U2-Pad29): track 0.00 -> 5.11 mm
- net Net-(U2-Pad21): track 0.00 -> 5.11 mm
- net Net-(U2-Pad51): track 0.00 -> 2.55 mm
- net Net-(U2-Pad25): track 0.00 -> 2.55 mm
- net Net-(U2-Pad19): track 0.00 -> 2.55 mm
- net Net-(U2-Pad11): track 0.00 -> 2.55 mm
- net Net-(U2-Pad49): track 0.00 -> 2.55 mm
- net Net-(U2-Pad43): track 0.00 -> 2.55 mm
- net Net-(U2-Pad41): track 0.00 -> 2.55 mm
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
Commit message: Main board traced
Parts:
- moved U2 64.4 mm to (58.4, 23.6)
- moved T2 59.4 mm to (10.9, 46.2), turned to 0 degrees
- moved D9 34.0 mm to (1.88, 64.0)
- moved D10 11.1 mm to (29.7, 81.8)
- moved C1 9.41 mm to (30.2, 46.6)
- moved C3 7.69 mm to (21.1, 46.5)
- moved D1 4.55 mm to (47.6, 81.8)
- moved D2 4.55 mm to (45.3, 81.8)
- moved D3 4.29 mm to (43.1, 81.8)
- moved D4 3.79 mm to (40.9, 81.8)
- moved C2 3.30 mm to (27.1, 46.7)
- moved D5 3.30 mm to (38.6, 81.8)
- moved R19 2.91 mm to (23.4, 47.4), turned to 180 degrees
- moved D6 2.81 mm to (36.4, 81.8)
- moved D7 2.12 mm to (34.2, 81.8)
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Connections:
- J2 pad 2: Net-(J1-Pad2) -> unconnected-(J2-Pad2)
- J2 pad 3: Net-(J1-Pad3) -> unconnected-(J2-Pad3)
- J2 pad 4: Net-(J1-Pad4) -> unconnected-(J2-Pad4)
- U2 pad 16: Net-(U2-Pad13) -> unconnected-(U2-Pad16)
- U2 pad 24: Net-(U2-Pad21) -> unconnected-(U2-Pad24)
- U2 pad 32: Net-(U2-Pad29) -> unconnected-(U2-Pad32)
- U2 pad 8: VCC -> unconnected-(U2-Pad8)
Routing:
- net GND: track 17.8 -> 345.3 mm, vias 0 -> 9
- net VCC: track 15.3 -> 261.8 mm, vias 0 -> 4
- net Net-(D10-Pad2): track 0.00 -> 162.4 mm, vias 0 -> 1
- net Net-(R26-Pad2): track 0.00 -> 135.3 mm, vias 0 -> 2
- net Net-(D9-Pad2): track 0.00 -> 132.2 mm, vias 0 -> 1
- net Net-(R1-Pad1): track 0.00 -> 129.6 mm, vias 0 -> 2
- net /7: track 0.00 -> 122.2 mm, vias 0 -> 1
- net Net-(D10-Pad1): track 0.00 -> 111.9 mm
- net /12(MISO): track 0.00 -> 110.5 mm
- net /13(SCK): track 0.00 -> 108.2 mm
- net Net-(D9-Pad1): track 0.00 -> 104.5 mm
- net /8: track 0.00 -> 101.9 mm, vias 0 -> 2
- net /0(Rx): track 0.00 -> 101.0 mm
- net /1(Tx): track 0.00 -> 92.6 mm, vias 0 -> 1
- net Net-(R_reset_pullup1-Pad2): track 0.00 -> 82.1 mm, vias 0 -> 1
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Other:
- board text added: "12 Drawing 13 Memory 14 Music 15 Media Player 16 Metronome 17 Sequencer 18 Notes 19 Composer 20 Noise 21 Hacker 22 Baby"
- board text removed: "12 Drawing 13 Memory 14 Music 15 Media 16 Metronome 17 Sequencer 18 Notes 19 Composer 20 Noise 21 Hacker 22 Baby"
