File: pcb/Luciebox_v5/button_pcb/button_pcb.kicad_sch (KiCad schematic)
At the start: 23 parts, among them T1 terminal_8x1, T2 terminal_8x1, T3 terminal_8x1, T4 terminal_2x1, U1 8X8PADS

Commit message: Start pcb v5 with feedback from v4
Connections:
- net at U1.25: no longer U1.26
- net at U1.27: no longer U1.28
- net at U1.30, U1.31, U1.32: no longer U1.29
- net at U1.33: no longer U1.34
- net at U1.35: no longer U1.36
- net at U1.38, U1.39, U1.40: no longer U1.37
- net at U1.41: no longer U1.42
- net at U1.43: no longer U1.44
- net at U1.46, U1.47, U1.48: no longer U1.45
- net at U1.49: no longer U1.50
- net at U1.51: no longer U1.52
- net at U1.54, U1.55, U1.56: no longer U1.53

Commit message: Pcb V5
Parts:
- removed H1, H2, H3, H4: MountingHole, Luciebox_components:MountingHole_4.3mm_M4, symbol Luciebox_components:MountingHole
- removed U1: 8X8PADS, Luciebox_components:8X8PADS_100mil, symbol Luciebox_components:8X8PADS
- added JPowerBankAsBattery1: USB_B_Mini, Luciebox_components:usb_mini_Molex-0548190519, symbol Luciebox_components:USB_B_Mini
- S1, S2, S3, S4: footprint Luciebox_components:button_LAZ16-11_big_holes -> Luciebox_components:button_square_17.5x17.5mm_big_holes; symbol Luciebox_components:button_laz16-11 -> Luciebox_components:button_square
Connections:
- net at BT1.2 (-), T1.4, T4.1: now also JPowerBankAsBattery1.1 (GND), JPowerBankAsBattery1.6 (Shield)
- net at BT1.1 (+), T1.5, T4.2: now also JPowerBankAsBattery1.5 (VBUS)
Other:
- moved on the sheet: BT1, H5, H6, H7, H8, S1, S2, S3, S4, S5, S6, S7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
